Commit message: added rviz config

File: bumperbot_ws/src/bumperbot_description/urdf/bumperbot_description.urdf (robot description, URDF)
Before this commit: robot bumperbot_description, 7 links, 6 joints
Links:
- added link base_footprint
Joints:
- added joint base_joint: type fixed, parent base_footprint, child base_link, origin xyz=0.0 0.0 0.033 rpy=0 0 0

Commit message: updated description

File: bumperbot_ws/src/bumperbot_description/urdf/bumperbot_description.urdf (robot description, URDF)
Before this commit: robot bumperbot_description, 8 links, 7 joints
Links:
- removed link base_footprint
- added link imu_link, mass 0.000528415362211671; collision mesh filename=package://bumperbot_description/meshes/imu_link.STL; visual mesh filename=package://bumperbot_description/meshes/imu_link.STL
- link base_link: mass 0.0913060531508687 -> 0.091306007508054
- link camera_link: mass 0.0041086 -> 0.0041086489783227
- link caster_front_link: mass 4.5247E-07 -> 1.44379265037903E-06
- link caster_rear_link: mass 4.5247E-07 -> 1.44379265037902E-06
- link laser_link: mass 0 -> 0.073084435549317
- link wheel_left_link: mass 0.053009 -> 0.0530086043219396
- link wheel_right_link: mass 0.053009 -> 0.053008609096452
Joints:
- removed joint base_joint
- added joint imu_joint: type fixed, parent base_link, child imu_link, origin xyz=0 0 0.069899 rpy=3.1416 0 0, axis 0 0 0
- joint camera_joint: origin xyz=0.040774 -0.0135 0.081 rpy=1.5708 0 -3.1416 -> xyz=0.081561 0 0.067457 rpy=0 -0.23739 0
- joint caster_front_joint: axis 0 0 1 -> 0 0 0; origin xyz=0.042791 0.00016909 -0.024363 rpy=1.5708 0 -1.6063 -> xyz=0.04755 0 -0.025363 rpy=0 0 0
- joint caster_rear_joint: axis 0 0 1 -> 0 0 0; origin xyz=-0.042791 -0.00016909 -0.024363 rpy=1.5708 0 -1.6063 -> xyz=-0.04755 0 -0.025363 rpy=0 0 0
- joint laser_joint: origin xyz=-0.0877495976327923 -0.140414680218275 -0.640692319552455 rpy=1.5707963267949 0 -3.08450753931019 -> xyz=-0.0050526 -0.0023221 0.1208 rpy=0 0 0
- joint wheel_left_joint: origin xyz=0 0.07011 0 rpy=1.5708 0.26876 -3.1416 -> xyz=0 0.07011 0 rpy=1.5708 0.36986 3.1416
- joint wheel_right_joint: origin xyz=0 -0.07011 0 rpy=-1.5708 -1.0554 3.1416 -> xyz=0 -0.07011 0 rpy=-1.5708 -0.95428 3.1416

Commit message: Fix URDF frames

File: bumperbot_ws/src/bumperbot_description/urdf/bumperbot_description.urdf (robot description, URDF)
Before this commit: robot description, 8 links, 7 joints
Links:
- added link base_footprint
Joints:
- added joint base_joint: type fixed, parent base_footprint, child base_link, origin xyz=0 0 0.033 rpy=0 0 0
- joint caster_front_joint: origin xyz=0.04755 0 -0.025363 rpy=0 0 0 -> xyz=0.04755 0 -0.0285 rpy=0 0 0
- joint caster_rear_joint: origin xyz=-0.04755 0 -0.025363 rpy=0 0 0 -> xyz=-0.04755 0 -0.0285 rpy=0 0 0
