Commit message: updated wheel rotation axis

File: bumperbot_ws/src/bumperbot_description/urdf/bumperbot.urdf (robot description, URDF)
Before this commit: robot description, 8 links, 7 joints
Links:
- link laser_link: mass 0.073084435549317 -> 0.0730844355551672
- link wheel_left_link: mass 0.0530086043219396 -> 0.0530086043217644
- link wheel_right_link: mass 0.053008609096452 -> 0.0530086090966721
Joints:
- joint imu_joint: origin xyz=0 0 0.069899 rpy=3.1416 0 0 -> xyz=0 0 0.0698986241758014 rpy=3.14159265358979 0 0
- joint wheel_right_joint: origin xyz=0 -0.07011 0 rpy=-1.5708 -0.95428 3.1416 -> xyz=0 -0.0701101849418637 0 rpy=1.5707963267949 0 -3.14159265358979

Commit message: updated wheels

File: bumperbot_ws/src/bumperbot_description/urdf/bumperbot.urdf (robot description, URDF)
Before this commit: robot bumperbot, 8 links, 8 joints
Links:
- added link base_footprint
- link laser_link: mass 0.0730844355551672 -> 0.073084435549317
Joints:
- joint caster_front_joint: origin xyz=0.04755 0 -0.0285 rpy=0 0 0 -> xyz=0.04755 0 -0.025363 rpy=0 0 0
- joint caster_rear_joint: origin xyz=-0.04755 0 -0.0285 rpy=0 0 0 -> xyz=-0.04755 0 -0.025363 rpy=0 0 0
- joint wheel_left_joint: axis 0 0 1 -> 0 1 0; origin xyz=0 0.07011 0 rpy=1.5708 0.36986 3.1416 -> xyz=0 0.0701101849418642 0 rpy=0 0 0
- joint wheel_right_joint: axis 0 0 1 -> 0 -1 0; origin xyz=0 -0.0701101849418637 0 rpy=1.5707963267949 0 -3.14159265358979 -> xyz=0 -0.0701101849418637 0 rpy=0 0 0

Commit message: added gazebo properties and controller

File: bumperbot_ws/src/bumperbot_description/urdf/bumperbot.urdf (robot description, URDF)
Before this commit: robot bumperbot, 9 links, 8 joints
Joints:
- joint caster_front_joint: origin xyz=0.04755 0 -0.025363 rpy=0 0 0 -> xyz=0.04755 0 -0.027 rpy=0 0 0
- joint caster_rear_joint: origin xyz=-0.04755 0 -0.025363 rpy=0 0 0 -> xyz=-0.04755 0 -0.027 rpy=0 0 0
- joint wheel_right_joint: axis 0 -1 0 -> 0 1 0
