Commit message: small fixes and formatting

File: bumperbot_ws/src/bumperbot_description/urdf/bumperbot_ros2_control.xacro (robot description, xacro)
@@ -2,5 +2,4 @@
 <robot xmlns:xacro="http://www.ros.org/wiki/xacro" name="bumperbot">
     <ros2_control name="RobotSystem" type="system">
-        <xacro:property name="PI" value="3.14159265359" />
         <!-- ros2_control Gazebo -->
         <xacro:if value="$(arg is_sim)">
