Commit message: finetuning gazebo model

File: bumperbot_ws/src/bumperbot_description/urdf/bumperbot.urdf.xacro (robot description, xacro)
@@ -5,5 +5,5 @@
   <link name="base_link">
     <inertial>
-      <origin xyz="0 0 0" rpy="0 0 0" />
+      <origin xyz="0 0 0.04" rpy="0.0 0.65 0.3" />
       <mass value="8.2573504e-01"/>
       <inertia ixx="2.2124416e-03" ixy="-1.2294101e-05" ixz="3.4938785e-05"
@@ -34,5 +34,5 @@
   <link name="wheel_right_link">
     <inertial>
-      <origin xyz="0 0 0" rpy="0 0 0" />
+      <origin xyz="0 -0.014 0" rpy="0 0 0" />
       <mass value="0.0530086090966721" />
       <inertia ixx="1.88176298336665E-05" ixy="-4.8444933029987E-10" ixz="1.88163708851143E-08"
@@ -65,5 +65,5 @@
     name="wheel_left_link">
     <inertial>
-      <origin xyz="0.000216638831504246 0.0137052653316193 -0.000640606107818048" rpy="0 0 0" />
+      <origin xyz="0 0.014 0" rpy="0 0 0" />
       <mass value="0.0530086043217644" />
       <inertia ixx="1.8792911368909E-05"  ixy="3.31256392204584E-10" ixz="-1.14082001662767E-08"
@@ -113,5 +113,5 @@
       <origin xyz="0 0 0" rpy="0 0 0" />
       <geometry>
-        <box size="0.030 0.020 0.008"/>
+        <box size="0.030 0.020 0.0095"/>
       </geometry>
     </collision>
@@ -143,5 +143,5 @@
       <origin xyz="0 0 0" rpy="0 0 0" />
       <geometry>
-        <box size="0.030 0.020 0.008"/>
+        <box size="0.030 0.020 0.0095"/>
       </geometry>
     </collision>

File: bumperbot_ws/src/bumperbot_description/urdf/bumperbot_gazebo.xacro (robot description, xacro)
@@ -26,7 +26,7 @@
     </transmission>
     <gazebo reference="wheel_left_link">
-      <mu1>1000000.0</mu1>
-      <mu2>1000000.0</mu2>
-      <kp>500000.0</kp>
+      <mu1>1000000000.0</mu1>
+      <mu2>1000000000.0</mu2>
+      <kp>1000000.0</kp>
       <kd>10.0</kd>
       <minDepth>0.001</minDepth>
@@ -36,7 +36,7 @@
     </gazebo>
     <gazebo reference="wheel_right_link">
-      <mu1>1000000.0</mu1>
-      <mu2>1000000.0</mu2>
-      <kp>500000.0</kp>
+      <mu1>1000000000.0</mu1>
+      <mu2>1000000000.0</mu2>
+      <kp>1000000.0</kp>
       <kd>10.0</kd>
       <minDepth>0.001</minDepth>

Commit message: finetuning controller parameters

File: bumperbot_ws/src/bumperbot_description/urdf/bumperbot.urdf.xacro (robot description, xacro)
@@ -5,9 +5,9 @@
   <link name="base_link">
     <inertial>
-      <origin xyz="0 0 0.04" rpy="0.0 0.65 0.3" />
+      <origin xyz="0 0 0.04" rpy="0.0 0.25 0.3" />
       <mass value="8.2573504e-01"/>
-      <inertia ixx="2.2124416e-03" ixy="-1.2294101e-05" ixz="3.4938785e-05"
-               iyy="2.1193702e-03" iyz="-5.0120904e-06"
-               izz="2.0064271e-03" />
+      <inertia ixx="2.2124416e-02" ixy="-1.2294101e-04" ixz="3.4938785e-04"
+               iyy="2.1193702e-02" iyz="-5.0120904e-05"
+               izz="2.0064271e-02" />
     </inertial>
     <visual>
@@ -52,5 +52,5 @@
       <origin xyz="0 -0.015 0" rpy="1.57 0 0" />
       <geometry>
-        <cylinder length="0.027" radius="0.033"/>
+        <sphere radius="0.033"/>
       </geometry>
     </collision>
@@ -83,5 +83,5 @@
       <origin xyz="0 0.015 0" rpy="-1.57 0 0" />
       <geometry>
-        <cylinder length="0.027" radius="0.033"/>
+        <sphere radius="0.033"/>
       </geometry>
     </collision>
@@ -113,5 +113,5 @@
       <origin xyz="0 0 0" rpy="0 0 0" />
       <geometry>
-        <box size="0.030 0.020 0.0095"/>
+        <sphere radius="0.005"/>
       </geometry>
     </collision>
@@ -143,5 +143,5 @@
       <origin xyz="0 0 0" rpy="0 0 0" />
       <geometry>
-        <box size="0.030 0.020 0.0095"/>
+        <sphere radius="0.005"/>
       </geometry>
     </collision>

File: bumperbot_ws/src/bumperbot_description/urdf/bumperbot_gazebo.xacro (robot description, xacro)
@@ -26,7 +26,7 @@
     </transmission>
     <gazebo reference="wheel_left_link">
-      <mu1>1000000000.0</mu1>
-      <mu2>1000000000.0</mu2>
-      <kp>1000000.0</kp>
+      <mu1>1000000000000000.0</mu1>
+      <mu2>1000000000000000.0</mu2>
+      <kp>1000000000000.0</kp>
       <kd>10.0</kd>
       <minDepth>0.001</minDepth>
@@ -36,7 +36,7 @@
     </gazebo>
     <gazebo reference="wheel_right_link">
-      <mu1>1000000000.0</mu1>
-      <mu2>1000000000.0</mu2>
-      <kp>1000000.0</kp>
+      <mu1>1000000000000000.0</mu1>
+      <mu2>1000000000000000.0</mu2>
+      <kp>1000000000000.0</kp>
       <kd>10.0</kd>
       <minDepth>0.001</minDepth>

Commit message: added imu republisher node and kalman filter

File: bumperbot_ws/src/bumperbot_description/urdf/bumperbot.urdf.xacro (robot description, xacro)
@@ -243,5 +243,5 @@
   </link>
   <joint name="imu_joint" type="fixed">
-    <origin xyz="0 0 0.0698986241758014" rpy="3.14159265358979 0 0" />
+    <origin xyz="0 0 0.0698986241758014" rpy="0 0 0" />
     <parent link="base_link" />
     <child link="imu_link" />

File: bumperbot_ws/src/bumperbot_description/urdf/bumperbot_gazebo.xacro (robot description, xacro)
@@ -114,12 +114,5 @@
             </linear_acceleration>
           </imu>
-          <plugin name="imu" filename="libgazebo_ros_imu_sensor.so">
-              <ros>
-                  <namespace>imu</namespace>
-                  <remapping>~/out:=data</remapping>
-              </ros>
-              <initial_orientation_as_reference>false</initial_orientation_as_reference>
-              <frame_name>imu_link</frame_name>
-          </plugin>
+          <plugin name="imu" filename="libgazebo_ros_imu_sensor.so"/>
       </sensor>
   </gazebo>

Commit message: uniform with course lessons

File: bumperbot_ws/src/bumperbot_description/urdf/bumperbot.urdf.xacro (robot description, xacro)
@@ -1,6 +1,4 @@
 <?xml version="1.0"?>
 <robot name="bumperbot" xmlns:xacro="http://ros.org/wiki/xacro">
-  <!-- Load Simulated or Real Hardware Interfaces -->
-  <xacro:arg name="is_sim" default="true"/>
   <!-- Include Gazebo Parameters -->
   <xacro:include filename="$(find bumperbot_description)/urdf/bumperbot_gazebo.xacro" />
@@ -21,7 +19,4 @@
         <mesh filename="package://bumperbot_description/meshes/base_link.STL" />
       </geometry>
-      <material name="">
-        <color rgba="0.258823529411765 0.27843137254902 0.301960784313725 1" />
-      </material>
     </visual>
     <collision>
@@ -50,7 +45,4 @@
         <mesh filename="package://bumperbot_description/meshes/wheel_right_link.STL" />
       </geometry>
-      <material name="">
-        <color rgba="0.831372549019608 0.670588235294118 0.129411764705882 1" />
-      </material>
     </visual>
     <collision>
@@ -81,7 +73,4 @@
         <mesh filename="package://bumperbot_description/meshes/wheel_left_link.STL" />
       </geometry>
-      <material name="">
-        <color rgba="0.792156862745098 0.819607843137255 0.933333333333333 1" />
-      </material>
     </visual>
     <collision>
@@ -111,7 +100,4 @@
         <mesh filename="package://bumperbot_description/meshes/caster_front_link.STL" />
       </geometry>
-      <material name="">
-        <color rgba="1 0 0 1" />
-      </material>
     </visual>
     <collision>
@@ -141,7 +127,4 @@
         <mesh filename="package://bumperbot_description/meshes/caster_rear_link.STL" />
       </geometry>
-      <material name="">
-        <color rgba="0.258823529411765 0.27843137254902 0.301960784313725 1" />
-      </material>
     </visual>
     <collision>
@@ -156,64 +139,4 @@
     <parent link="base_link" />
     <child link="caster_rear_link" />
-    <axis xyz="0 0 0" />
-  </joint>
-  <link name="camera_link">
-    <inertial>
-      <origin xyz="-0.0122943599302166 -9.05173297049283E-07 0.00843684900384606" rpy="0 0 0" />
-      <mass value="0.0041086489783227" />
-      <inertia ixx="3.98797447678453E-07" ixy="-8.24558929781979E-11" ixz="1.22069699665359E-07"
-               iyy="4.18205575812023E-07" iyz="-1.01562924198144E-10"
-               izz="4.28578734986182E-07" />
-    </inertial>
-    <visual>
-      <origin xyz="0 0 0" rpy="0 0 0" />
-      <geometry>
-        <mesh filename="package://bumperbot_description/meshes/camera_link.STL" />
-      </geometry>
-      <material name="">
-        <color rgba="0.792156862745098 0.819607843137255 0.933333333333333 1" />
-      </material>
-    </visual>
-    <collision>
-      <origin xyz="0 0 0" rpy="0 0 0" />
-      <geometry>
-        <mesh filename="package://bumperbot_description/meshes/camera_link.STL" />
-      </geometry>
-    </collision>
-  </link>
-  <joint name="camera_joint" type="fixed">
-    <origin xyz="0.081561 0 0.067457" rpy="0 -0.23739 0" />
-    <parent link="base_link" />
-    <child link="camera_link" />
-    <axis xyz="0 0 0" />
-  </joint>
-  <link name="laser_link">
-    <inertial>
-      <origin xyz="-0.011945780406062 -0.000381929217680526 -0.0170649378129477" rpy="0 0 0" />
-      <mass value="0.073084435549317" />
-      <inertia ixx="1.96074931730795E-05" ixy="-3.62091076640009E-07" ixz="4.28230084046735E-07"
-               iyy="2.40983835136327E-05" iyz="1.50180909250652E-08"
-               izz="4.14184164228595E-05" />
-    </inertial>
-    <visual>
-      <origin xyz="0 0 0" rpy="0 0 0" />
-      <geometry>
-        <mesh filename="package://bumperbot_description/meshes/laser_link.STL" />
-      </geometry>
-      <material name="">
-        <color rgba="0.792156862745098 0.819607843137255 0.933333333333333 1" />
-      </material>
-    </visual>
-    <collision>
-      <origin xyz="0 0 0" rpy="0 0 0" />
-      <geometry>
-        <mesh filename="package://bumperbot_description/meshes/laser_link.STL" />
-      </geometry>
-    </collision>
-  </link>
-  <joint name="laser_joint" type="fixed">
-    <origin xyz="-0.0050526 -0.0023221 0.1208" rpy="0 0 0" />
-    <parent link="base_link" />
-    <child link="laser_link" />
     <axis xyz="0 0 0" />
   </joint>

File: bumperbot_ws/src/bumperbot_description/urdf/bumperbot_gazebo.xacro (robot description, xacro)
@@ -1,119 +1,112 @@
 <?xml version="1.0"?>
 <robot name="bumperbot" xmlns:xacro="http://ros.org/wiki/xacro">
-    <gazebo reference="base_link">
-      <material>Gazebo/DarkGrey</material>
-    </gazebo>
-    <!-- Move this one to ros2 control -->
-    <transmission name="wheel_right_transmission">
-      <plugin>transmission_interface/SimpleTransmission</plugin>
-      <actuator name="wheel_right_motor" role="actuator_right"/>
-      <joint name="wheel_right_joint"    role="joint_right">
-        <mechanical_reduction>1.0</mechanical_reduction>
-      </joint>
-    </transmission>
-    <transmission name="wheel_left_transmission">
-      <plugin>transmission_interface/SimpleTransmission</plugin>
-      <actuator name="wheel_left_motor" role="actuator_left"/>
-      <joint name="wheel_left_joint"    role="joint_left">
-        <mechanical_reduction>1.0</mechanical_reduction>
-      </joint>
-    </transmission>
-    <!-- Wheels -->
-    <gazebo reference="wheel_left_link">
-      <mu1>1000000000000000.0</mu1>
-      <mu2>1000000000000000.0</mu2>
-      <kp>1000000000000.0</kp>
-      <kd>10.0</kd>
-      <minDepth>0.001</minDepth>
-      <maxVel>0.1</maxVel>
-      <fdir1>1 0 0</fdir1>
-      <material>Gazebo/Blue</material>
-    </gazebo>
-    <gazebo reference="wheel_right_link">
-      <mu1>1000000000000000.0</mu1>
-      <mu2>1000000000000000.0</mu2>
-      <kp>1000000000000.0</kp>
-      <kd>10.0</kd>
-      <minDepth>0.001</minDepth>
-      <maxVel>0.1</maxVel>
-      <fdir1>1 0 0</fdir1>
-      <material>Gazebo/Blue</material>
-    </gazebo>
-    <!-- Caster Wheels -->
-    <gazebo reference="caster_rear_link">
-      <mu1>0.1</mu1>
-      <mu2>0.1</mu2>
-      <kp>1000000.0</kp>
-      <kd>100.0</kd>
-      <minDepth>0.001</minDepth>
-      <maxVel>1.0</maxVel>
-      <material>Gazebo/FlatBlack</material>
-    </gazebo>
-    <gazebo reference="caster_front_link">
-      <mu1>0.1</mu1>
-      <mu2>0.1</mu2>
-      <kp>1000000.0</kp>
-      <kd>100.0</kd>
-      <minDepth>0.001</minDepth>
-      <maxVel>1.0</maxVel>
-      <material>Gazebo/FlatBlack</material>
-    </gazebo>
-    <!-- ROS Control -->
-    <gazebo>
-      <plugin filename="libgazebo_ros2_control.so" name="gazebo_ros2_control">
-        <robot_param>robot_description</robot_param>
-        <robot_param_node>robot_state_publisher</robot_param_node>
-        <parameters>$(find bumperbot_controller)/config/bumperbot_controllers.yaml</parameters>
-      </plugin>
-    </gazebo>
-    <!-- IMU -->
-    <gazebo reference="imu_link">
-      <sensor name="imu" type="imu">
-          <always_on>true</always_on>
-          <update_rate>100</update_rate>
-          <imu>
-            <angular_velocity>
-              <x>
-                <noise type="gaussian">
-                  <mean>0.0</mean>
-                  <stddev>2e-4</stddev>
-                </noise>
-              </x>
-              <y>
-                <noise type="gaussian">
-                  <mean>0.0</mean>
-                  <stddev>2e-4</stddev>
-                </noise>
-              </y>
-              <z>
-                <noise type="gaussian">
-                  <mean>0.0</mean>
-                  <stddev>2e-4</stddev>
-                </noise>
-              </z>
-            </angular_velocity>
-            <linear_acceleration>
-              <x>
-                <noise type="gaussian">
-                  <mean>0.0</mean>
-                  <stddev>1.7e-2</stddev>
-                </noise>
-              </x>
-              <y>
-                <noise type="gaussian">
-                  <mean>0.0</mean>
-                  <stddev>1.7e-2</stddev>
-                </noise>
-              </y>
-              <z>
-                <noise type="gaussian">
-                  <mean>0.0</mean>
-                  <stddev>1.7e-2</stddev>
-                </noise>
-              </z>
-            </linear_acceleration>
-          </imu>
-          <plugin name="imu" filename="libgazebo_ros_imu_sensor.so"/>
-      </sensor>
+  <!-- Move this one to ros2 control -->
+  <transmission name="wheel_right_transmission">
+    <plugin>transmission_interface/SimpleTransmission</plugin>
+    <actuator name="wheel_right_motor" role="actuator_right"/>
+    <joint name="wheel_right_joint"    role="joint_right">
+      <mechanical_reduction>1.0</mechanical_reduction>
+    </joint>
+  </transmission>
+  <transmission name="wheel_left_transmission">
+    <plugin>transmission_interface/SimpleTransmission</plugin>
+    <actuator name="wheel_left_motor" role="actuator_left"/>
+    <joint name="wheel_left_joint"    role="joint_left">
+      <mechanical_reduction>1.0</mechanical_reduction>
+    </joint>
+  </transmission>
+  <!-- Wheels -->
+  <gazebo reference="wheel_left_link">
+    <mu1>1000000000000000.0</mu1>
+    <mu2>1000000000000000.0</mu2>
+    <kp>1000000000000.0</kp>
+    <kd>10.0</kd>
+    <minDepth>0.001</minDepth>
+    <maxVel>0.1</maxVel>
+    <fdir1>1 0 0</fdir1>
+  </gazebo>
+  <gazebo reference="wheel_right_link">
+    <mu1>1000000000000000.0</mu1>
+    <mu2>1000000000000000.0</mu2>
+    <kp>1000000000000.0</kp>
+    <kd>10.0</kd>
+    <minDepth>0.001</minDepth>
+    <maxVel>0.1</maxVel>
+    <fdir1>1 0 0</fdir1>
+  </gazebo>
+  <!-- Caster Wheels -->
+  <gazebo reference="caster_rear_link">
+    <mu1>0.1</mu1>
+    <mu2>0.1</mu2>
+    <kp>1000000.0</kp>
+    <kd>100.0</kd>
+    <minDepth>0.001</minDepth>
+    <maxVel>1.0</maxVel>
+  </gazebo>
+  <gazebo reference="caster_front_link">
+    <mu1>0.1</mu1>
+    <mu2>0.1</mu2>
+    <kp>1000000.0</kp>
+    <kd>100.0</kd>
+    <minDepth>0.001</minDepth>
+    <maxVel>1.0</maxVel>
+  </gazebo>
+  <!-- ROS 2 Control -->
+  <gazebo>
+    <plugin filename="libgazebo_ros2_control.so" name="gazebo_ros2_control">
+      <robot_param>robot_description</robot_param>
+      <robot_param_node>robot_state_publisher</robot_param_node>
+      <parameters>$(find bumperbot_controller)/config/bumperbot_controllers.yaml</parameters>
+    </plugin>
+  </gazebo>
+  <!-- IMU -->
+  <gazebo reference="imu_link">
+    <sensor name="imu" type="imu">
+        <always_on>true</always_on>
+        <update_rate>100</update_rate>
+        <imu>
+          <angular_velocity>
+            <x>
+              <noise type="gaussian">
+                <mean>0.0</mean>
+                <stddev>2e-4</stddev>
+              </noise>
+            </x>
+            <y>
+              <noise type="gaussian">
+                <mean>0.0</mean>
+                <stddev>2e-4</stddev>
+              </noise>
+            </y>
+            <z>
+              <noise type="gaussian">
+                <mean>0.0</mean>
+                <stddev>2e-4</stddev>
+              </noise>
+            </z>
+          </angular_velocity>
+          <linear_acceleration>
+            <x>
+              <noise type="gaussian">
+                <mean>0.0</mean>
+                <stddev>1.7e-2</stddev>
+              </noise>
+            </x>
+            <y>
+              <noise type="gaussian">
+                <mean>0.0</mean>
+                <stddev>1.7e-2</stddev>
+              </noise>
+            </y>
+            <z>
+              <noise type="gaussian">
+                <mean>0.0</mean>
+                <stddev>1.7e-2</stddev>
+              </noise>
+            </z>
+          </linear_acceleration>
+        </imu>
+        <plugin name="imu" filename="libgazebo_ros_imu_sensor.so"/>
+    </sensor>
   </gazebo>
 </robot>

File: bumperbot_ws/src/bumperbot_description/urdf/bumperbot_ros2_control.xacro (robot description, xacro)
@@ -3,16 +3,7 @@
     <ros2_control name="RobotSystem" type="system">
         <!-- ros2_control Gazebo -->
-        <xacro:if value="$(arg is_sim)">
-            <hardware>
-                <plugin>gazebo_ros2_control/GazeboSystem</plugin>
-            </hardware>
-        </xacro:if>
-        <!-- ros2_control Real Robot -->
-        <xacro:unless value="$(arg is_sim)">
-            <hardware>
-                <plugin>bumperbot_controller/BumperbotInterface</plugin>
-                <param name="port">/dev/ttyACM0</param>
-            </hardware>
-        </xacro:unless>
+        <hardware>
+            <plugin>gazebo_ros2_control/GazeboSystem</plugin>
+        </hardware>
         <!-- ros2_control Common Interfaces -->
         <joint name="wheel_right_joint">

Commit message: gazebo world, odometry motion model

File: bumperbot_ws/src/bumperbot_description/urdf/bumperbot.urdf.xacro (robot description, xacro)
@@ -156,7 +156,4 @@
         <mesh filename="package://bumperbot_description/meshes/imu_link.STL" />
       </geometry>
-      <material name="">
-        <color rgba="0.792156862745098 0.819607843137255 0.933333333333333 1" />
-      </material>
     </visual>
     <collision>
@@ -173,3 +170,30 @@
     <axis xyz="0 0 0" />
   </joint>
+  <link name="laser_link">
+    <inertial>
+      <origin xyz="-0.011945780406062 -0.000381929217680526 -0.0170649378129477" rpy="0 0 0" />
+      <mass value="0.073084435549317" />
+      <inertia ixx="1.96074931730795E-05" ixy="-3.62091076640009E-07" ixz="4.28230084046735E-07"
+               iyy="2.40983835136327E-05" iyz="1.50180909250652E-08"
+               izz="4.14184164228595E-05" />
+    </inertial>
+    <visual>
+      <origin xyz="0 0 0" rpy="0 0 0" />
+      <geometry>
+        <mesh filename="package://bumperbot_description/meshes/laser_link.STL" />
+      </geometry>
+    </visual>
+    <collision>
+      <origin xyz="0 0 0" rpy="0 0 0" />
+      <geometry>
+        <mesh filename="package://bumperbot_description/meshes/laser_link.STL" />
+      </geometry>
+    </collision>
+  </link>
+  <joint name="laser_joint" type="fixed">
+    <origin xyz="-0.0050526 -0.0023221 0.1208" rpy="0 0 0" />
+    <parent link="base_link" />
+    <child link="laser_link" />
+    <axis xyz="0 0 0" />
+  </joint>
 </robot>

Commit message: init mapping with known poses

File: bumperbot_ws/src/bumperbot_description/urdf/bumperbot.urdf.xacro (robot description, xacro)
@@ -11,5 +11,5 @@
     <inertial>
       <origin xyz="0 0 0.04" rpy="0.0 0.25 0.3" />
-      <mass value="8.2573504e-01"/>
+      <mass value="1.0"/>
       <inertia ixx="2.2124416e-02" ixy="-1.2294101e-04" ixz="3.4938785e-04"
                iyy="2.1193702e-02" iyz="-5.0120904e-05"
@@ -37,5 +37,5 @@
     <inertial>
       <origin xyz="0 -0.014 0" rpy="0 0 0" />
-      <mass value="0.0530086090966721" />
+      <mass value="1.0" />
       <inertia ixx="1.88176298336665E-05" ixy="-4.8444933029987E-10" ixz="1.88163708851143E-08"
                iyy="3.11510738647764E-05" iyz="-6.93560663069607E-11"
@@ -65,5 +65,5 @@
     <inertial>
       <origin xyz="0 0.014 0" rpy="0 0 0" />
-      <mass value="0.0530086043217644" />
+      <mass value="1.0" />
       <inertia ixx="1.8792911368909E-05"  ixy="3.31256392204584E-10" ixz="-1.14082001662767E-08"
                iyy="3.11510738759073E-05" iyz="-3.60499245082192E-10"
